Commit message: 0.1.0-alpha release

File: assets/hanger.urdf (robot description, URDF)
Before this commit: robot hanger, 2 links, 1 joints
Links:
- added link branch_base, mass .0; collision cylinder length=0.03 radius=0.007; visual cylinder length=0.03 radius=0.007
- link base_link: geometry collision box size=0.01 0.03 0.3; visual box size=0.01 0.03 0.3
- link branch: geometry collision cylinder length=0.07 radius=0.007; visual cylinder length=0.07 radius=0.007
Joints:
- added joint base_to_branch_base: type fixed, parent base_link, child branch_base, origin xyz=0.0 0 0.21 rpy=0 1.5707963267948966 0
- joint base_to_branch: origin xyz=0 0 0.15 rpy=0 0.60 0 -> xyz=0.0 0 0.03 rpy=0 -1.0471975511965976 0; parent base_link -> branch_base
